File: amplifier_board.kicad_pcb (KiCad board)
At the start: 2 copper layers, 125.7 x 83.8 mm, 72 parts, among them J1 external input, J10 external saw, J11 jumper storage, J2 AUDIO, J3 VCC, J4 +5V, J5 GND, J6 -5V, J7 audio tune, J8 speaker, J9 speaker, Q1 SQJ860EP, Q2 Q_NMOS_GSD, Q3 SQJ860EP, U1 AD8038, U2 AD8613, U3 LTC4444-5, U4 AD8468, U5 LM555, U6 AD8038, U7 AD8613

Commit message: up
Parts:
- moved C22 43.8 mm to (65.2, 34.8), turned to 0 degrees
- moved C23 34.3 mm to (69.1, 30.7)
Connections:
- C22 pad 2: -5V -> +5V
- C23 pad 2: -5V -> +5V
Routing:
- net +5V: track 235.5 -> 257.6 mm
- net -5V: track 114.9 -> 136.6 mm
- net GND: track 419.4 -> 438.1 mm
Changed lines of the file:
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@@
     (thickness 1.6)
     (drawings 4)
-    (tracks 548)
+    (tracks 579)
     (zones 0)
     (modules 72)
@@
   )
   (module Capacitors_SMD:C_1206_HandSoldering (layer F.Cu)
-    (at 83.852 -0.254)
+    (at 69.056 30.734)
     (descr "Capacitor SMD 1206, hand soldering")
     (tags "capacitor 1206")
@@
       (net 5 GND))
     (pad 2 smd rect (at 2 0) (size 2 1.6) (layers F.Cu F.Paste F.Mask)
-      (net 9 -5V))
+      (net 8 +5V))
     (model Capacitors_SMD.3dshapes/C_1206.wrl
       (at (xyz 0 0 0))
@@
   )
   (module Capacitors_SMD:C_1206_HandSoldering (layer F.Cu)
-    (at 83.312 -5.08 180)
+    (at 65.246 34.798)
     (descr "Capacitor SMD 1206, hand soldering")
     (tags "capacitor 1206")
     (attr smd)
-    (fp_text reference C22 (at 0 -1.75 180) (layer F.SilkS)
+    (fp_text reference C22 (at 0 -1.75) (layer F.SilkS)
       (effects (font (size 1 1) (thickness 0.15)))
     )
-    (fp_text value 100nF (at 0 2 180) (layer F.Fab)
+    (fp_text value 100nF (at 0 2) (layer F.Fab)
       (effects (font (size 1 1) (thickness 0.15)))
     )
@@
     (fp_line (start 1.6 0.8) (end -1.6 0.8) (layer F.Fab) (width 0.1))
     (fp_line (start -1.6 0.8) (end -1.6 -0.8) (layer F.Fab) (width 0.1))
-    (fp_text user %R (at 0 -1.75 180) (layer F.Fab)
+    (fp_text user %R (at 0 -1.75) (layer F.Fab)
       (effects (font (size 1 1) (thickness 0.15)))
     )
-    (pad 2 smd rect (at 2 0 180) (size 2 1.6) (layers F.Cu F.Paste F.Mask)
-      (net 9 -5V))
-    (pad 1 smd rect (at -2 0 180) (size 2 1.6) (layers F.Cu F.Paste F.Mask)
+    (pad 2 smd rect (at 2 0) (size 2 1.6) (layers F.Cu F.Paste F.Mask)
+      (net 8 +5V))
+    (pad 1 smd rect (at -2 0) (size 2 1.6) (layers F.Cu F.Paste F.Mask)
       (net 5 GND))
     (model Capacitors_SMD.3dshapes/C_1206.wrl
@@
   (segment (start 24.13 24.13) (end 16.510001 31.749999) (width 5) (layer F.Cu) (net 5))
   (segment (start 17.78 46.99) (end 17.78 45.212) (width 2) (layer F.Cu) (net 5))
-  (segment (start 54.61 38.118693) (end 64.77 27.958693) (width 5) (layer F.Cu) (net 5))
   (segment (start 54.61 48.895) (end 54.61 38.118693) (width 5) (layer F.Cu) (net 5))
   (segment (start 64.77 27.958693) (end 64.77 22.86) (width 5) (layer F.Cu) (net 5))
@@
   (segment (start 14.10001 46.35199) (end 14.10001 67.44001) (width 2) (layer F.Cu) (net 5))
   (segment (start 101.092 64.008) (end 101.092 62.992) (width 1) (layer F.Cu) (net 5))
+  (segment (start 56.388 35.894) (end 56.388 36.340693) (width 2) (layer F.Cu) (net 5))
+  (segment (start 55.292 34.798) (end 56.388 35.894) (width 2) (layer F.Cu) (net 5))
+  (segment (start 52.292 34.798) (end 55.292 34.798) (width 2) (layer F.Cu) (net 5))
+  (segment (start 54.61 38.118693) (end 56.388 36.340693) (width 5) (layer F.Cu) (net 5))
+  (segment (start 60.594 31.75) (end 60.978693 31.75) (width 2) (layer F.Cu) (net 5))
+  (segment (start 59.578 30.734) (end 60.594 31.75) (width 2) (layer F.Cu) (net 5))
+  (segment (start 56.578 30.734) (end 59.578 30.734) (width 2) (layer F.Cu) (net 5))
+  (segment (start 56.388 36.340693) (end 60.978693 31.75) (width 5) (layer F.Cu) (net 5))
+  (segment (start 60.978693 31.75) (end 64.77 27.958693) (width 5) (layer F.Cu) (net 5))
+  (segment (start 67.056 30.244693) (end 64.77 27.958693) (width 2) (layer F.Cu) (net 5))
+  (segment (start 67.056 30.734) (end 67.056 30.244693) (width 2) (layer F.Cu) (net 5))
+  (segment (start 62.998 31.75) (end 60.978693 31.75) (width 2) (layer F.Cu) (net 5))
+  (segment (start 63.246 31.998) (end 62.998 31.75) (width 2) (layer F.Cu) (net 5))
+  (segment (start 63.246 34.798) (end 63.246 31.998) (width 2) (layer F.Cu) (net 5))
   (segment (start 71.306049 67.276958) (end 70.711049 66.681958) (width 1) (layer F.Cu) (net 6))
   (segment (start 73.841049 67.276958) (end 71.306049 67.276958) (width 1) (layer F.Cu) (net 6))
@@
   (segment (start 63.969999 43.286855) (end 76.835 30.421854) (width 5) (layer F.Cu) (net 8))
   (segment (start 63.969999 43.345001) (end 63.969999 43.286855) (width 5) (layer F.Cu) (net 8))
-  (segment (start 74.93 32.385) (end 63.969999 43.345001) (width 5) (layer F.Cu) (net 8))
   (segment (start 74.93 28.516854) (end 74.93 32.385) (width 5) (layer F.Cu) (net 8))
   (segment (start 88.9 67.904) (end 90.129 66.675) (width 1) (layer F.Cu) (net 8))
@@
   (segment (start 120.512 66.908) (end 121.412 66.008) (width 2) (layer F.Cu) (net 8))
   (segment (start 117.856 66.908) (end 120.512 66.908) (width 2) (layer F.Cu) (net 8))
+  (segment (start 67.246 40.069) (end 66.802 40.513) (width 2) (layer F.Cu) (net 8))
+  (segment (start 67.246 34.798) (end 67.246 40.069) (width 2) (layer F.Cu) (net 8))
+  (segment (start 74.93 32.385) (end 66.802 40.513) (width 5) (layer F.Cu) (net 8))
+  (segment (start 66.802 40.513) (end 63.969999 43.345001) (width 5) (layer F.Cu) (net 8))
+  (segment (start 74.93 31.608) (end 74.93 32.385) (width 2) (layer F.Cu) (net 8))
+  (segment (start 74.056 30.734) (end 74.93 31.608) (width 2) (layer F.Cu) (net 8))
+  (segment (start 71.056 30.734) (end 74.056 30.734) (width 2) (layer F.Cu) (net 8))
+  (segment (start 67.564 15.494) (end 74.93 22.86) (width 2) (layer F.Cu) (net 8))
+  (segment (start 66.77 15.494) (end 67.564 15.494) (width 2) (layer F.Cu) (net 8))
   (segment (start 41.18 36.29) (end 41.18 55.88) (width 5) (layer F.Cu) (net 9))
-  (segment (start 54.61 22.86) (end 41.18 36.29) (width 5) (layer F.Cu) (net 9))
   (segment (start 41.18 64.135) (end 41.18 55.88) (width 1) (layer F.Cu) (net 9))
   (segment (start 38.900011 64.914989) (end 39.68 64.135) (width 0.5) (layer F.Cu) (net 9))
@@
   (segment (start 53.975 75.86) (end 57.109 78.994) (width 2) (layer F.Cu) (net 9))
   (segment (start 53.975 75.66) (end 53.975 75.86) (width 2) (layer F.Cu) (net 9))
+  (segment (start 48.768 29.924) (end 48.768 28.702) (width 2) (layer F.Cu) (net 9))
+  (segment (start 49.578 30.734) (end 48.768 29.924) (width 2) (layer F.Cu) (net 9))
+  (segment (start 52.578 30.734) (end 49.578 30.734) (width 2) (layer F.Cu) (net 9))
+  (segment (start 54.61 22.86) (end 48.768 28.702) (width 5) (layer F.Cu) (net 9))
+  (segment (start 44.53 34.036) (end 43.434 34.036) (width 2) (layer F.Cu) (net 9))
+  (segment (start 45.292 34.798) (end 44.53 34.036) (width 2) (layer F.Cu) (net 9))
+  (segment (start 48.292 34.798) (end 45.292 34.798) (width 2) (layer F.Cu) (net 9))
+  (segment (start 48.768 28.702) (end 43.434 34.036) (width 5) (layer F.Cu) (net 9))
+  (segment (start 43.434 34.036) (end 41.18 36.29) (width 5) (layer F.Cu) (net 9))
+  (segment (start 61.976 15.494) (end 54.61 22.86) (width 2) (layer F.Cu) (net 9))
+  (segment (start 62.77 15.494) (end 61.976 15.494) (width 2) (layer F.Cu) (net 9))
   (segment (start 85.09 28.516854) (end 83.185 30.421854) (width 5) (layer F.Cu) (net 10))
   (segment (start 85.09 22.86) (end 85.09 28.516854) (width 5) (layer F.Cu) (net 10))

Commit message: more files
Parts:
- added C24: 100nF, Capacitor_SMD:C_1206_3216Metric_Pad1.42x1.75mm_HandSolder, F.Cu at (69.8, 88.7)
- added C25: 100nF, Capacitor_SMD:C_1206_3216Metric_Pad1.42x1.75mm_HandSolder, F.Cu at (73.2, 88.9)
- added JP4: internal audio, Connector_PinHeader_2.54mm:PinHeader_1x02_P2.54mm_Vertical, F.Cu at (63.5, 68.6)
Connections:
- J11 pad 1: (no net) -> Net-(J11-Pad1)
- J11 pad 2: (no net) -> Net-(J11-Pad2)
- J11 pad 3: (no net) -> Net-(J11-Pad3)
- J11 pad 4: (no net) -> Net-(J11-Pad4)
- J11 pad 5: (no net) -> Net-(J11-Pad5)
- J11 pad 6: (no net) -> Net-(J11-Pad6)
- R7 pad 1: /audio -> Net-(JP4-Pad1)
- U1 pad 1: (no net) -> Net-(U1-Pad1)
- U1 pad 5: (no net) -> Net-(U1-Pad5)
- U1 pad 6: /audio -> Net-(JP4-Pad1)
- U1 pad 8: (no net) -> Net-(U1-Pad8)
- U4 pad 5: (no net) -> Net-(U4-Pad5)
- U5 pad 3: (no net) -> Net-(U5-Pad3)
- U6 pad 1: (no net) -> Net-(U6-Pad1)
- U6 pad 5: (no net) -> Net-(U6-Pad5)
- U6 pad 8: (no net) -> Net-(U6-Pad8)
Routing:
- net +5V: track 257.6 -> 313.7 mm
- net -5V: track 136.6 -> 183.6 mm
- net /audio: track 94.7 -> 59.2 mm
- net Net-(JP4-Pad1): track 0.00 -> 30.1 mm
- net GND: track 438.1 -> 413.9 mm, vias 2 -> 1
- net Net-(J1-Pad1): track 60.7 -> 70.9 mm
- net Net-(C1-Pad2): track 73.5 -> 81.7 mm
- net Net-(R14-Pad2): track 25.0 -> 22.2 mm
- net Net-(JP2-Pad1): track 9.24 -> 10.0 mm
- net Net-(R11-Pad1): track 12.6 -> 13.4 mm
