File: amplifier_board.kicad_pcb (KiCad board)
At the start: 2 copper layers, 57 parts, among them J1 VCC (7-14V), J2 AUDIO, J3 GND, J4 speaker, J8 speaker, Q1 SQJ860EP, Q2 Q_NMOS_GSD, Q3 SQJ860EP, U1 AD8038, U2 AD8613, U3 LTC4444-5, U4 AD8468, U5 L7805, U6 LM2776, U7 AD8038, U8 AD8468

Commit message: pcb
Parts:
- removed C1: large, Capacitors_ThroughHole:CP_Radial_D10.0mm_P2.50mm_P5.00mm
- removed C3: 100uF, Capacitors_SMD:C_1206_HandSoldering
- removed J8: speaker, Terminal_Blocks:TerminalBlock_bornier-2_P5.08mm
- removed R1, R2: 220, Resistors_SMD:R_1206_HandSoldering
- added D4: Schottky, Diodes_SMD:D_SMA-SMB_Universal_Handsoldering, F.Cu at (163.2, 94.0)
- added D5: Schottky, Diodes_SMD:D_SMA-SMB_Universal_Handsoldering, F.Cu at (172.1, 96.5)
- added D6: Schottky, Diodes_SMD:D_SMA-SMB_Universal_Handsoldering, F.Cu at (172.1, 74.3)
- added J5: B, Wire_Pads:SolderWirePad_single_SMD_5x10mm, F.Cu at (191.1, 54.6)
- added JP1: Jumper-Device, Pin_Headers:Pin_Header_Straight_1x02_Pitch2.54mm, F.Cu at (157.2, 72.5)
- added JP3: Jumper-Device, Pin_Headers:Pin_Header_Straight_1x02_Pitch2.54mm, F.Cu at (157.2, 68.5)
- added L2: 10uH, Choke_Toroid_ThroughHole:Choke_Toroid_8x16mm_Vertical, F.Cu at (176.5, 77.5)
- added Q4: SQJ402EP, SMD_Packages:SO-8_PowerPAK_Vishay_Single, F.Cu at (172.1, 90.2)
- added Q5: SQJ402EP, SMD_Packages:SO-8_PowerPAK_Vishay_Single, F.Cu at (172.0, 80.6)
- added U9: LTC4444-5, Housings_SSOP:MSOP-8-1EP_3x3mm_Pitch0.65mm, F.Cu at (163.4, 83.4)
- C7: value 100uF -> 1.5uF
- C8: value 100uF -> 2.2uF
- J1, J3: footprint Mounting_Holes:MountingHole_4mm_Pad -> Wire_Pads:SolderWirePad_single_SMD_5x10mm
- J2: footprint Pin_Headers:Pin_Header_Straight_1x03_Pitch2.54mm -> Pin_Headers:Pin_Header_Angled_1x02_Pitch2.54mm
- J4: value speaker -> A; footprint Pin_Headers:Pin_Header_Straight_1x02_Pitch2.54mm -> Wire_Pads:SolderWirePad_single_SMD_5x10mm
- Q1, Q3: value SQJ860EP -> SQJ402EP
- moved C4 169.0 mm to (190.5, 107.3), turned to 270 degrees
- moved C2 158.8 mm to (183.5, 106.7), turned to 90 degrees
- moved U5 152.6 mm to (179.2, 106.0)
- moved C21 150.0 mm to (171.8, 110.4)
- moved C10 140.9 mm to (165.6, 109.7), turned to 90 degrees
- moved J1 136.1 mm to (190.5, 98.4), turned to 90 degrees
- moved J3 111.9 mm to (190.5, 71.1), turned to 90 degrees
- moved C9 96.4 mm to (186.7, 61.6), turned to 270 degrees
- moved R6 91.9 mm to (125.1, 103.4), turned to 90 degrees
- moved C11 90.8 mm to (155.6, 107.3), turned to 180 degrees
- moved JP2 90.5 mm to (141.6, 92.8)
- moved C7 90.0 mm to (186.7, 78.7), turned to 90 degrees
- moved R8 89.9 mm to (127.0, 108.0)
- moved J2 89.7 mm to (134.7, 75.8)
- moved C19 89.7 mm to (145.7, 103.8)
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Connections:
- C5 pad 1: Net-(C1-Pad2) -> Net-(C5-Pad1)
- C5 pad 2: Net-(C1-Pad1) -> Net-(C5-Pad2)
- C7 pad 1: Net-(C1-Pad2) -> Net-(C7-Pad1)
- C7 pad 2: Net-(C1-Pad1) -> GND
- C8 pad 1: Net-(C1-Pad2) -> GND
- C8 pad 2: Net-(C1-Pad1) -> Net-(C8-Pad2)
- C9 pad 1: Net-(C1-Pad1) -> Net-(C9-Pad1)
- J2 pad 2: Net-(J2-Pad2) -> /audio_in
- J4 pad 1: Net-(C1-Pad2) -> Net-(C7-Pad1)
- L1 pad 2: Net-(C1-Pad1) -> Net-(C9-Pad1)
- Q2 pad 1: Net-(Q2-Pad1) -> Net-(JP1-Pad1)
- Q2 pad 3: Net-(Q2-Pad3) -> Net-(JP3-Pad1)
- R12 pad 1: Net-(Q2-Pad3) -> Net-(JP3-Pad1)
- RV3 pad 2: Net-(RV3-Pad2) -> Net-(C8-Pad2)
- U3 pad 1: Net-(Q2-Pad1) -> Net-(JP1-Pad2)
- U3 pad 2: Net-(Q2-Pad3) -> Net-(JP3-Pad2)
- U4 pad 1: Net-(Q2-Pad1) -> Net-(JP1-Pad1)
- U7 pad 3: Net-(RV3-Pad2) -> Net-(C8-Pad2)
- U8 pad 4: Net-(RV3-Pad2) -> Net-(C8-Pad2)
Routing:
- net GND: track 51.3 -> 364.0 mm, vias 0 -> 2
- net VCC: track 0.00 -> 187.1 mm, vias 0 -> 3
- net Net-(C6-Pad1): track 0.00 -> 82.0 mm
- net Net-(C5-Pad1): track 0.00 -> 51.6 mm
- net Net-(JP3-Pad2): track 0.00 -> 27.5 mm
- net Net-(JP1-Pad2): track 0.00 -> 26.5 mm
- net Net-(Q1-Pad4): track 0.00 -> 25.7 mm
- net Net-(JP1-Pad1): track 0.00 -> 22.3 mm
- net Net-(C8-Pad2): track 0.00 -> 17.5 mm
- net Net-(RV3-Pad2): track 17.2 -> 0.00 mm
- net Net-(C6-Pad2): track 0.00 -> 16.4 mm
- net Net-(C9-Pad1): track 0.00 -> 13.8 mm
- net Net-(Q4-Pad4): track 0.00 -> 12.7 mm
- net +5V: track 109.6 -> 122.2 mm
- net Net-(C7-Pad1): track 0.00 -> 12.3 mm
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Other:
- net class Default: via_dia 0.8 -> 2; via_drill 0.4 -> 1
- rule via_min_drill: 0.3 -> 1
- rule via_min_size: 0.4 -> 1.8

Commit message: pcb ready
Parts:
- moved C4 37.0 mm to (154.6, 98.4)
- moved U5 37.0 mm to (143.3, 97.2)
- moved C2 37.0 mm to (147.6, 97.8)
- moved C10 35.6 mm to (135.8, 90.3)
- moved C21 32.9 mm to (140.5, 100.3)
- moved C13 29.7 mm to (125.3, 97.8), turned to 180 degrees
- moved C14 28.4 mm to (120.7, 95.8), turned to 90 degrees
- moved U6 24.7 mm to (123.7, 93.9), turned to 90 degrees
- moved C12 23.4 mm to (129.8, 82.0), turned to 90 degrees
- moved R5 22.4 mm to (126.1, 64.7)
- moved R7 22.4 mm to (128.1, 76.8)
- moved C17 22.4 mm to (131.2, 66.7)
- moved C20 22.4 mm to (136.2, 79.9)
- moved JP2 22.4 mm to (136.8, 71.0)
- moved R3 22.4 mm to (129.3, 61.7)
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Routing:
- net +5V: track 122.2 -> 168.8 mm, vias 0 -> 4
- net -5V: track 42.8 -> 86.3 mm
- net GND: track 364.0 -> 395.3 mm, vias 2 -> 4
- net Net-(JP1-Pad1): track 22.3 -> 9.90 mm
- net Net-(C8-Pad2): track 17.5 -> 25.7 mm
- net /audio_in: track 15.5 -> 8.06 mm
- net Net-(R9-Pad2): track 5.87 -> 10.1 mm
- net /audio: track 5.30 -> 8.72 mm
- net /sawtooth: track 6.05 -> 8.88 mm
- net VCC: track 187.1 -> 186.0 mm
- net Net-(RV1-Pad2): track 4.59 -> 4.02 mm

Commit message: pcb improvements
Parts:
- added RV4: 5k, Pin_Headers:Pin_Header_Straight_1x03_Pitch2.54mm, F.Cu at (116.5, 82.2)
- moved C18 6.41 mm to (150.7, 71.6), turned to 180 degrees
- moved R6 4.14 mm to (124.2, 80.4), turned to 0 degrees
- moved C14 3.08 mm to (117.7, 95.1)
- moved Q2 2.65 mm to (153.3, 64.9)
- moved R12 2.65 mm to (150.7, 69.2)
- moved U4 2.65 mm to (148.8, 65.3)
- moved R4 2.59 mm to (119.6, 82.1)
- moved R3 2.45 mm to (127.3, 60.2), turned to 180 degrees
- moved R8 2.40 mm to (124.2, 87.4)
- moved U6 2.34 mm to (121.4, 94.2)
- moved C15 2.18 mm to (120.9, 90.4)
- moved C13 2.16 mm to (125.2, 95.6), turned to 90 degrees
- moved U2 2.16 mm to (124.2, 84.1)
- moved R5 1.99 mm to (127.3, 63.1), turned to 180 degrees
- moved J2 1.89 mm to (134.4, 59.7)
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Connections:
- J2 pad 1: GND -> /audio_in
- J2 pad 2: /audio_in -> GND
- R8 pad 1: Net-(R6-Pad1) -> Net-(R8-Pad1)
- U2 pad 3: Net-(R6-Pad1) -> Net-(RV4-Pad2)
Routing:
- net GND: track 395.3 -> 372.3 mm, vias 4 -> 2
- net +5V: track 168.8 -> 159.1 mm
- net Net-(RV4-Pad2): track 0.00 -> 7.19 mm
- net -5V: track 86.3 -> 93.2 mm
- net Net-(R8-Pad1): track 0.00 -> 5.83 mm
- net Net-(R3-Pad2): track 15.5 -> 11.4 mm
- net Net-(C19-Pad1): track 20.1 -> 24.0 mm
- net Net-(R4-Pad2): track 10.9 -> 7.27 mm
- net /audio_in: track 8.06 -> 5.23 mm
- net /sawtooth: track 8.88 -> 10.7 mm
- net Net-(R4-Pad1): track 6.80 -> 8.36 mm
- net /audio: track 8.72 -> 10.3 mm
- net Net-(JP3-Pad1): track 9.13 -> 10.5 mm
- net Net-(R5-Pad2): track 6.14 -> 5.19 mm
- net Net-(R6-Pad1): track 8.03 -> 7.31 mm
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
Commit message: better inverter
Parts:
- removed C15: 1uF, Capacitors_SMD:C_1206_HandSoldering
- removed U6: LM2776, TO_SOT_Packages_SMD:SOT-23-6_Handsoldering
- added C1: 2.2uF, Capacitors_SMD:C_1206_HandSoldering, F.Cu at (134.5, 63.2)
- added C22: 2.2uF, Capacitors_SMD:C_1206_HandSoldering, F.Cu at (130.4, 92.5)
- added C23: 2.2uF, Capacitors_SMD:C_1206_HandSoldering, F.Cu at (115.8, 97.7)
- added C24: 1.5uF, Capacitors_SMD:C_1206_HandSoldering, F.Cu at (122.8, 99.7)
- added C26: 2.2uF, Capacitors_SMD:C_1206_HandSoldering, F.Cu at (120.3, 90.9)
- added C3: 2.2uF, Capacitors_SMD:C_1206_HandSoldering, F.Cu at (128.3, 92.5)
- added D7: LED, LEDs:LED_1206_HandSoldering, F.Cu at (132.8, 100.2)
- added D8: LED, LEDs:LED_1206_HandSoldering, F.Cu at (113.5, 97.7)
- added J6: 5V, Pin_Headers:Pin_Header_Straight_1x02_Pitch2.54mm, F.Cu at (127.4, 102.2)
- added J7: -5v, Pin_Headers:Pin_Header_Straight_1x02_Pitch2.54mm, F.Cu at (125.7, 64.1)
- added R1: 2k2, Resistors_SMD:R_1206_HandSoldering, F.Cu at (128.3, 97.2)
- added R10: 200k, Resistors_SMD:R_1206_HandSoldering, F.Cu at (118.1, 97.7)
- added R11: 50k, Resistors_SMD:R_1206_HandSoldering, F.Cu at (117.1, 102.2)
- added R2: 2k2, Resistors_SMD:R_1206_HandSoldering, F.Cu at (113.5, 91.1)
- added U10: LM27761, Housings_DFN_QFN:VDFN-8-1EP_2x2mm_Pitch0.5mm, F.Cu at (121.7, 96.5)
- C10, C4: value large -> 470uF; footprint Capacitors_ThroughHole:CP_Radial_D10.0mm_P2.50mm_P5.00mm -> Capacitors_SMD:CP_Elec_8x10
- C11, C2: value 100nF -> 1uF
- C12, C17, C18, C20, C21: value 100nF -> 2.2uF
- C5, C6: value 100uF -> 1.5uF
- U5: footprint TO_SOT_Packages_THT:TO-220-3_Vertical -> TO_SOT_Packages_SMD:TO-252-2_Rectifier
- moved C21 21.2 mm to (154.4, 84.3)
- moved C2 13.2 mm to (160.4, 100.7)
- moved C11 13.0 mm to (137.7, 97.9), turned to 180 degrees
- moved J2 8.13 mm to (128.0, 54.6), turned to 0 degrees
- moved R3 5.46 mm to (122.3, 58.0)
- moved C13 3.30 mm to (126.1, 92.5)
- moved C14 3.25 mm to (120.3, 93.1), turned to 180 degrees
- moved D4 1.94 mm to (162.8, 92.1)
- moved R5 1.91 mm to (127.3, 61.2)
- moved U5 1.65 mm to (144.9, 97.2), turned to 270 degrees
- moved C10 1.20 mm to (136.9, 89.9)
- moved C16 0.63 mm to (160.3, 83.6)
- moved C4 0.28 mm to (154.4, 98.7)
Connections:
- C14 pad 2: -5V -> Net-(C14-Pad2)
Routing:
- net GND: track 372.3 -> 402.8 mm
- net +5V: track 159.1 -> 170.3 mm
- net -5V: track 93.2 -> 100.3 mm
- net Net-(R10-Pad1): track 0.00 -> 6.83 mm
- net Net-(C14-Pad2): track 0.00 -> 6.79 mm
- net Net-(R3-Pad2): track 11.4 -> 7.54 mm
- net Net-(C24-Pad1): track 0.00 -> 3.24 mm
- net Net-(D7-Pad2): track 0.00 -> 2.97 mm
- net Net-(C15-Pad1): track 2.95 -> 0.00 mm
- net Net-(C15-Pad2): track 2.86 -> 0.00 mm
- net Net-(C24-Pad2): track 0.00 -> 2.65 mm
- net Net-(D8-Pad1): track 0.00 -> 2.60 mm
- net VCC: track 186.0 -> 187.6 mm
- net /audio_in: track 5.23 -> 6.19 mm
- net Net-(JP4-Pad1): track 15.3 -> 14.4 mm
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Other:
- board outline added: 87 x 63.5 mm
- board text added: "Jan Równicki Wzmacniacz klasy D"

Commit message: plan B for output filter
Parts:
- added C15: 1uF, Capacitors_SMD:C_1206_HandSoldering, F.Cu at (193.0, 78.8)
- added C27: 1uF, Capacitors_SMD:C_1206_HandSoldering, F.Cu at (190.5, 76.2)
- added C28: 1uF, Capacitors_SMD:C_1206_HandSoldering, F.Cu at (193.0, 61.0)
- added C29: 1uF, Capacitors_SMD:C_1206_HandSoldering, F.Cu at (190.5, 63.5)
- C11, C2: value 1uF -> 2.2uF
- C24, C5, C6, C7, C9: value 1.5uF -> 1uF
- moved C9 1.42 mm to (188.0, 61.0)
- moved C7 1.27 mm to (188.0, 78.7)
- moved J3 1.27 mm to (190.5, 69.8)
Routing:
- net GND: track 402.8 -> 424.9 mm
- net Net-(C15-Pad1): track 12.3 -> 17.1 mm
- net Net-(C28-Pad1): track 13.8 -> 17.8 mm
- net Net-(C28-Pad2): track 0.00 -> 3.14 mm
- net Net-(C15-Pad2): track 0.00 -> 3.11 mm

Commit message: final?
Parts:
- added C30: 2.2uF, Capacitors_SMD:C_1206_HandSoldering, F.Cu at (162.7, 100.7)
- R11, R4, R7: value 50k -> 68k
- R12, R8: value 10k -> 11k
- moved C19 3.39 mm to (138.5, 79.5), turned to 0 degrees
- moved C1 3.18 mm to (137.5, 62.4), turned to 270 degrees
- moved C20 2.17 mm to (137.1, 81.9)
- moved L1 0.90 mm to (177.2, 47.6)
- moved L2 0.65 mm to (177.2, 77.6)
- moved J4 0.63 mm to (191.1, 85.1)
- moved R9 0.54 mm to (145.6, 76.1)
- moved U7 0.41 mm to (137.6, 75.6)
- moved R7 0.19 mm to (128.3, 76.8)
Routing:
- net +5V: track 170.3 -> 148.9 mm
- net -5V: track 100.3 -> 89.6 mm
- net GND: track 424.9 -> 417.8 mm
- net Net-(C19-Pad1): track 24.0 -> 28.7 mm
- net Net-(R9-Pad2): track 10.1 -> 9.29 mm

Commit message: text and small fixes
Parts:
- moved C1 0.23 mm to (137.6, 62.1)
- moved J2 0.21 mm to (128.1, 54.4)
- moved C10 0.20 mm to (136.7, 89.9)
Routing:
- net Net-(C6-Pad1): track 82.0 -> 93.3 mm
- net VCC: track 187.6 -> 196.8 mm
- net Net-(Q3-Pad4): track 12.2 -> 17.4 mm
- net Net-(C5-Pad2): track 10.3 -> 7.73 mm
- net Net-(C6-Pad2): track 16.4 -> 18.6 mm
- net GND: track 417.8 -> 419.0 mm
Other:
- board text added: "-5"
- board text added: "5"
- board text added: "<-audio in"
- board text added: "GND"
- board text added: "Output A"
- board text added: "Output B"
- board text added: "PWr Openlab"
- board text added: "VCC"
- board text added: "amp"
- board text added: "audio"
- board text added: "driver input"
- board text added: "saw"
- board text added: "volume"

Commit message: fixes
Parts:
- moved C24 0.35 mm to (122.6, 99.4)
- moved R9 0.26 mm to (145.7, 75.8)
- moved J6 0.08 mm to (127.4, 102.3)
Routing:
- net Net-(C8-Pad2): track 25.7 -> 26.5 mm
Changed lines of the file:
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@@
     (thickness 1.6)
     (drawings 19)
-    (tracks 601)
+    (tracks 602)
     (zones 0)
     (modules 81)
@@
   )
   (setup
-    (last_trace_width 0.5)
+    (last_trace_width 1)
     (user_trace_width 0.35)
     (user_trace_width 0.4)
@@
     (add_net VCC)
   )
+  (module Resistors_SMD:R_1206_HandSoldering (layer F.Cu)
+    (at 145.6944 75.8444)
+    (descr "Resistor SMD 1206, hand soldering")
+    (tags "resistor 1206")
+    (attr smd)
+    (fp_text reference R9 (at 0 -1.85) (layer F.SilkS)
+      (effects (font (size 1 1) (thickness 0.15)))
+    )
+    (fp_text value 1k (at 0 1.9) (layer F.Fab)
+      (effects (font (size 1 1) (thickness 0.15)))
+    )
+    (fp_text user %R (at 0 0) (layer F.Fab)
+      (effects (font (size 0.7 0.7) (thickness 0.105)))
+    )
+    (fp_line (start -1.6 0.8) (end -1.6 -0.8) (layer F.Fab) (width 0.1))
+    (fp_line (start 1.6 0.8) (end -1.6 0.8) (layer F.Fab) (width 0.1))
+    (fp_line (start 1.6 -0.8) (end 1.6 0.8) (layer F.Fab) (width 0.1))
+    (fp_line (start -1.6 -0.8) (end 1.6 -0.8) (layer F.Fab) (width 0.1))
+    (fp_line (start 1 1.07) (end -1 1.07) (layer F.SilkS) (width 0.12))
+    (fp_line (start -1 -1.07) (end 1 -1.07) (layer F.SilkS) (width 0.12))
+    (fp_line (start -3.25 -1.11) (end 3.25 -1.11) (layer F.CrtYd) (width 0.05))
+    (fp_line (start -3.25 -1.11) (end -3.25 1.1) (layer F.CrtYd) (width 0.05))
+    (fp_line (start 3.25 1.1) (end 3.25 -1.11) (layer F.CrtYd) (width 0.05))
+    (fp_line (start 3.25 1.1) (end -3.25 1.1) (layer F.CrtYd) (width 0.05))
+    (pad 1 smd rect (at -2 0) (size 2 1.7) (layers F.Cu F.Paste F.Mask)
+      (net 6 "Net-(C19-Pad2)"))
+    (pad 2 smd rect (at 2 0) (size 2 1.7) (layers F.Cu F.Paste F.Mask)
+      (net 19 "Net-(R9-Pad2)"))
+    (model ${KISYS3DMOD}/Resistors_SMD.3dshapes/R_1206.wrl
+      (at (xyz 0 0 0))
+      (scale (xyz 1 1 1))
+      (rotate (xyz 0 0 0))
+    )
+  )
   (module Capacitors_SMD:C_1206_HandSoldering (layer F.Cu)
     (at 138.462 79.502)
@@
   )
   (module Resistors_SMD:R_1206_HandSoldering (layer F.Cu)
-    (at 145.574 76.073)
-    (descr "Resistor SMD 1206, hand soldering")
-    (tags "resistor 1206")
-    (attr smd)
-    (fp_text reference R9 (at 0 -1.85) (layer F.SilkS)
-      (effects (font (size 1 1) (thickness 0.15)))
-    )
-    (fp_text value 1k (at 0 1.9) (layer F.Fab)
-      (effects (font (size 1 1) (thickness 0.15)))
-    )
-    (fp_text user %R (at 0 0) (layer F.Fab)
-      (effects (font (size 0.7 0.7) (thickness 0.105)))
-    )
-    (fp_line (start -1.6 0.8) (end -1.6 -0.8) (layer F.Fab) (width 0.1))
-    (fp_line (start 1.6 0.8) (end -1.6 0.8) (layer F.Fab) (width 0.1))
-    (fp_line (start 1.6 -0.8) (end 1.6 0.8) (layer F.Fab) (width 0.1))
-    (fp_line (start -1.6 -0.8) (end 1.6 -0.8) (layer F.Fab) (width 0.1))
-    (fp_line (start 1 1.07) (end -1 1.07) (layer F.SilkS) (width 0.12))
-    (fp_line (start -1 -1.07) (end 1 -1.07) (layer F.SilkS) (width 0.12))
-    (fp_line (start -3.25 -1.11) (end 3.25 -1.11) (layer F.CrtYd) (width 0.05))
-    (fp_line (start -3.25 -1.11) (end -3.25 1.1) (layer F.CrtYd) (width 0.05))
-    (fp_line (start 3.25 1.1) (end 3.25 -1.11) (layer F.CrtYd) (width 0.05))
-    (fp_line (start 3.25 1.1) (end -3.25 1.1) (layer F.CrtYd) (width 0.05))
-    (pad 1 smd rect (at -2 0) (size 2 1.7) (layers F.Cu F.Paste F.Mask)
-      (net 6 "Net-(C19-Pad2)"))
-    (pad 2 smd rect (at 2 0) (size 2 1.7) (layers F.Cu F.Paste F.Mask)
-      (net 19 "Net-(R9-Pad2)"))
-    (model ${KISYS3DMOD}/Resistors_SMD.3dshapes/R_1206.wrl
-      (at (xyz 0 0 0))
-      (scale (xyz 1 1 1))
-      (rotate (xyz 0 0 0))
-    )
-  )
-  (module Resistors_SMD:R_1206_HandSoldering (layer F.Cu)
     (at 150.654 69.215 180)
     (descr "Resistor SMD 1206, hand soldering")
@@
   )
   (module Capacitors_SMD:C_1206_HandSoldering (layer F.Cu)
-    (at 122.841 99.695 180)
+    (at 122.6312 99.4156 180)
     (descr "Capacitor SMD 1206, hand soldering")
     (tags "capacitor 1206")
@@
   )
   (module Pin_Headers:Pin_Header_Straight_1x02_Pitch2.54mm (layer F.Cu)
-    (at 127.381 102.235 90)
+    (at 127.3556 102.3112 90)
     (descr "Through hole straight pin header, 1x02, 2.54mm pitch, single row")
     (tags "Through hole pin header THT 1x02 2.54mm single row")
@@
   (segment (start 147.26 81.982) (end 144.145 78.867) (width 0.5) (layer F.Cu) (net 19) (status 20))
   (segment (start 147.26 82.281) (end 147.26 81.982) (width 0.5) (layer F.Cu) (net 19) (status 10))
-  (segment (start 144.78 78.867) (end 147.574 76.073) (width 1) (layer F.Cu) (net 19))
-  (segment (start 144.145 78.867) (end 144.78 78.867) (width 1) (layer F.Cu) (net 19))
+  (segment (start 144.6718 78.867) (end 147.6944 75.8444) (width 1) (layer F.Cu) (net 19))
+  (segment (start 144.145 78.867) (end 144.6718 78.867) (width 1) (layer F.Cu) (net 19))
   (segment (start 146.319 83.581) (end 147.26 83.581) (width 0.5) (layer F.Cu) (net 20) (status 20))
   (segment (start 144.145 81.407) (end 146.319 83.581) (width 0.5) (layer F.Cu) (net 20) (status 10))
@@
   (segment (start 149.439999 86.780001) (end 148.59 87.63) (width 0.5) (layer F.Cu) (net 23))
   (segment (start 149.92 83.581) (end 149.92 84.281) (width 0.5) (layer F.Cu) (net 23))
-  (segment (start 141.923999 74.93) (end 140.335 74.93) (width 1) (layer F.Cu) (net 23))
-  (segment (start 142.281 74.572999) (end 141.923999 74.93) (width 1) (layer F.Cu) (net 23))
-  (segment (start 149.094001 74.422) (end 142.281 74.422) (width 1) (layer F.Cu) (net 23))
-  (segment (start 151.479 76.957998) (end 149.094001 74.572999) (width 1) (layer F.Cu) (net 23))
-  (segment (start 151.479 79.121) (end 151.479 76.957998) (width 1) (layer F.Cu) (net 23))
   (segment (start 149.92 83.581) (end 148.97 83.581) (width 0.2) (layer F.Cu) (net 23) (status 10))
   (segment (start 148.919999 81.480001) (end 148.993 81.407) (width 0.2) (layer F.Cu) (net 23))
@@
   (segment (start 151.279 79.121) (end 148.993 81.407) (width 0.5) (layer F.Cu) (net 23) (status 10))
   (segment (start 151.479 79.121) (end 151.279 79.121) (width 0.5) (layer F.Cu) (net 23) (status 30))
+  (segment (start 151.479 77.321) (end 151.479 79.121) (width 1) (layer F.Cu) (net 23))
+  (segment (start 151.479 76.608998) (end 151.479 77.321) (width 1) (layer F.Cu) (net 23))
+  (segment (start 141.310002 74.93) (end 142.427602 73.8124) (width 1) (layer F.Cu) (net 23))
+  (segment (start 140.335 74.93) (end 141.310002 74.93) (width 1) (layer F.Cu) (net 23))
+  (segment (start 148.682402 73.8124) (end 151.479 76.608998) (width 1) (layer F.Cu) (net 23))
+  (segment (start 142.427602 73.8124) (end 148.682402 73.8124) (width 1) (layer F.Cu) (net 23))
   (segment (start 149.494 63.948) (end 150.094 63.948) (width 0.4) (layer F.Cu) (net 24) (status 10))
   (segment (start 154.239 64.323) (end 157.226 67.31) (width 1) (layer F.Cu) (net 24))
