File: amplifier_board.sch (KiCad schematic (older format))
At the start: 63 parts, among them J1 VCC (7-14V), J2 AUDIO, J3 GND, J4 A, J5 B, Q1 SQJ402EP, Q2 Q_NMOS_GSD, Q3 SQJ402EP, Q4 SQJ402EP, Q5 SQJ402EP, U1 AD8038, U2 AD8613, U3 LTC4444-5, U4 AD8468, U5 L7805, U6 LM2776, U7 AD8038, U8 AD8468, U9 LTC4444-5

Commit message: better inverter
Parts:
- removed C15: 1uF, Capacitors_SMD:C_1206_HandSoldering, symbol amplifier_board-rescue:C-Device
- removed U6: LM2776, TO_SOT_Packages_SMD:SOT-23-6_Handsoldering, symbol Regulator_SwitchedCapacitor:LM2776
- added C1, C22, C23, C26, C3: 2.2uF, Capacitors_SMD:C_1206_HandSoldering, symbol amplifier_board-rescue:C-Device
- added C24: 1.5uF, Capacitors_SMD:C_1206_HandSoldering, symbol amplifier_board-rescue:C-Device
- added D7, D8: LED, LEDs:LED_1206_HandSoldering, symbol Device:LED
- added J6: 5V, Pin_Headers:Pin_Header_Straight_1x02_Pitch2.54mm, symbol Connector_Generic:Conn_01x02
- added J7: -5v, Pin_Headers:Pin_Header_Straight_1x02_Pitch2.54mm, symbol Connector_Generic:Conn_01x02
- added R1, R2: 2k2, Resistors_SMD:R_1206_HandSoldering, symbol amplifier_board-rescue:R-Device
- added R10: 200k, Resistors_SMD:R_1206_HandSoldering, symbol amplifier_board-rescue:R-Device
- added R11: 50k, Resistors_SMD:R_1206_HandSoldering, symbol amplifier_board-rescue:R-Device
- added U10: LM27761, Housings_DFN_QFN:VDFN-8-1EP_2x2mm_Pitch0.5mm, symbol Regulator_SwitchedCapacitor:LM27761
- C10, C4: value large -> 470uF; footprint Capacitors_ThroughHole:CP_Radial_D10.0mm_P2.50mm_P5.00mm -> Capacitors_SMD:CP_Elec_8x10
- C11, C12, C17, C18, C2, C20, C21: value 100nF -> 2.2uF
- C5, C6: value 100uF -> 1.5uF
- U5: footprint TO_SOT_Packages_THT:TO-220-3_Vertical -> TO_SOT_Packages_SMD:TO-252-2_Rectifier
Connections:
- net +5V: now also C22.1, C3.1, J6.1 (Pin_1), R1.2, U10.1 (VIN)
- net -5V: now also C1.2, C23.2, J7.2 (Pin_2), R10.2, R2.2, U10.4 (VOUT); no longer C14.2
- net GND: now also C1.1, C22.2, C23.1, C26.1, C3.2, D7.1 (K), D8.2 (A), J6.2 (Pin_2), J7.1 (Pin_1), R11.1, U10.2 (GND), U10.9 (PAD)
- new net: D7.2 (A), R1.1
- new net: D8.1 (K), R2.1
- new net: C14.2, C26.2, U10.3 (CPOUT)
- new net: R10.1, R11.2, U10.5 (VFB)
- new net: C24.2, U10.7 (C-)
- new net: C24.1, U10.8 (C+)
- no-connect marks 1 -> 0
Other:
- moved on the sheet: C12, C13, C14, C16, C17, C18, C19, C20, C21, C25, C5, C6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

Commit message: plan B for output filter
Parts:
- added C15, C27, C28, C29: 1uF, Capacitors_SMD:C_1206_HandSoldering, symbol amplifier_board-rescue:C-Device
- C24, C5, C6, C7, C9: value 1.5uF -> 1uF
Connections:
- net GND: now also C27.2, C29.2
- net at C9.1, J5.1 (Pin_1), L1.2: now also C28.1
- net at C7.1, J4.1 (Pin_1), L2.2: now also C15.1
- new net: C15.2, C27.1
- new net: C28.2, C29.1
Other:
- moved on the sheet: J4, J5
Changed lines of the file:
@@
 P 9650 4550
 F 0 "C9" H 9765 4596 50  0000 L CNN
-F 1 "1.5uF" H 9765 4505 50  0000 L CNN
+F 1 "1uF" H 9765 4505 50  0000 L CNN
 F 2 "Capacitors_SMD:C_1206_HandSoldering" H 9688 4400 50  0001 C CNN
 F 3 "~" H 9650 4550 50  0001 C CNN
@@
 P 8425 3925
 F 0 "C6" V 8300 3850 50  0000 C CNN
-F 1 "1.5uF" V 8300 4025 50  0000 C CNN
+F 1 "1uF" V 8300 4025 50  0000 C CNN
 F 2 "Capacitors_SMD:C_1206_HandSoldering" H 8463 3775 50  0001 C CNN
 F 3 "~" H 8425 3925 50  0001 C CNN
@@
 L Connector:Conn_01x01_Female J5
 U 1 1 5CCC2E4F
-P 10000 4400
-F 0 "J5" H 10028 4426 50  0000 L CNN
-F 1 "B" H 10028 4335 50  0000 L CNN
-F 2 "Wire_Pads:SolderWirePad_single_SMD_5x10mm" H 10000 4400 50  0001 C CNN
-F 3 "~" H 10000 4400 50  0001 C CNN
-	1    10000 4400
-	1    0    0    -1
-$EndComp
-Wire Wire Line
-	9650 4400 9800 4400
+P 10425 4400
+F 0 "J5" H 10453 4426 50  0000 L CNN
+F 1 "B" H 10453 4335 50  0000 L CNN
+F 2 "Wire_Pads:SolderWirePad_single_SMD_5x10mm" H 10425 4400 50  0001 C CNN
+F 3 "~" H 10425 4400 50  0001 C CNN
+	1    10425 4400
+	1    0    0    -1
+$EndComp
+Wire Wire Line
+	9650 4400 10100 4400
 Connection ~ 9650 4400
 $Comp
@@
 P 9700 3125
 F 0 "C7" H 9815 3171 50  0000 L CNN
-F 1 "1.5uF" H 9815 3080 50  0000 L CNN
+F 1 "1uF" H 9815 3080 50  0000 L CNN
 F 2 "Capacitors_SMD:C_1206_HandSoldering" H 9738 2975 50  0001 C CNN
 F 3 "~" H 9700 3125 50  0001 C CNN
@@
 P 8475 2500
 F 0 "C5" V 8350 2425 50  0000 C CNN
-F 1 "1.5uF" V 8350 2600 50  0000 C CNN
+F 1 "1uF" V 8350 2600 50  0000 C CNN
 F 2 "Capacitors_SMD:C_1206_HandSoldering" H 8513 2350 50  0001 C CNN
 F 3 "~" H 8475 2500 50  0001 C CNN
@@
 L Connector:Conn_01x01_Female J4
 U 1 1 5CCD8E39
-P 10050 2975
-F 0 "J4" H 10078 3001 50  0000 L CNN
-F 1 "A" H 10078 2910 50  0000 L CNN
-F 2 "Wire_Pads:SolderWirePad_single_SMD_5x10mm" H 10050 2975 50  0001 C CNN
-F 3 "~" H 10050 2975 50  0001 C CNN
-	1    10050 2975
-	1    0    0    -1
-$EndComp
-Wire Wire Line
-	9700 2975 9850 2975
+P 10425 2975
+F 0 "J4" H 10453 3001 50  0000 L CNN
+F 1 "A" H 10453 2910 50  0000 L CNN
+F 2 "Wire_Pads:SolderWirePad_single_SMD_5x10mm" H 10425 2975 50  0001 C CNN
+F 3 "~" H 10425 2975 50  0001 C CNN
+	1    10425 2975
+	1    0    0    -1
+$EndComp
+Wire Wire Line
+	9700 2975 10100 2975
 Connection ~ 9700 2975
 Wire Wire Line
@@
 P 4125 1400
 F 0 "C24" H 4000 1500 50  0000 L CNN
-F 1 "1.5uF" H 3925 1300 50  0000 L CNN
+F 1 "1uF" H 3925 1300 50  0000 L CNN
 F 2 "Capacitors_SMD:C_1206_HandSoldering" H 4163 1250 50  0001 C CNN
 F 3 "~" H 4125 1400 50  0001 C CNN
@@
 Wire Wire Line
 	1000 3400 1475 3400
+$Comp
+L amplifier_board-rescue:C-Device C15
+U 1 1 5CFA00C0
+P 10100 3125
+F 0 "C15" H 10215 3171 50  0000 L CNN
+F 1 "1uF" H 10215 3080 50  0000 L CNN
+F 2 "Capacitors_SMD:C_1206_HandSoldering" H 10138 2975 50  0001 C CNN
+F 3 "~" H 10100 3125 50  0001 C CNN
+	1    10100 3125
+	1    0    0    -1
+$EndComp
+Connection ~ 10100 2975
+Wire Wire Line
+	10100 2975 10225 2975
+$Comp
+L amplifier_board-rescue:C-Device C27
+U 1 1 5CFA01AA
+P 10100 3475
+F 0 "C27" H 10215 3521 50  0000 L CNN
+F 1 "1uF" H 10215 3430 50  0000 L CNN
+F 2 "Capacitors_SMD:C_1206_HandSoldering" H 10138 3325 50  0001 C CNN
+F 3 "~" H 10100 3475 50  0001 C CNN
+	1    10100 3475
+	1    0    0    -1
+$EndComp
+$Comp
+L amplifier_board-rescue:GND-power #PWR0136
+U 1 1 5CFA026A
+P 10100 3675
+F 0 "#PWR0136" H 10100 3425 50  0001 C CNN
+F 1 "GND" H 10105 3502 50  0000 C CNN
+F 2 "" H 10100 3675 50  0001 C CNN
+F 3 "" H 10100 3675 50  0001 C CNN
+	1    10100 3675
+	1    0    0    -1
+$EndComp
+Wire Wire Line
+	10100 3675 10100 3625
+Wire Wire Line
+	10100 3325 10100 3275
+$Comp
+L amplifier_board-rescue:C-Device C28
+U 1 1 5CFBC018
+P 10100 4550
+F 0 "C28" H 10215 4596 50  0000 L CNN
+F 1 "1uF" H 10215 4505 50  0000 L CNN
+F 2 "Capacitors_SMD:C_1206_HandSoldering" H 10138 4400 50  0001 C CNN
+F 3 "~" H 10100 4550 50  0001 C CNN
+	1    10100 4550
+	1    0    0    -1
+$EndComp
+$Comp
+L amplifier_board-rescue:C-Device C29
+U 1 1 5CFBC020
+P 10100 4900
+F 0 "C29" H 10215 4946 50  0000 L CNN
+F 1 "1uF" H 10215 4855 50  0000 L CNN
+F 2 "Capacitors_SMD:C_1206_HandSoldering" H 10138 4750 50  0001 C CNN
+F 3 "~" H 10100 4900 50  0001 C CNN
+	1    10100 4900
+	1    0    0    -1
+$EndComp
+$Comp
+L amplifier_board-rescue:GND-power #PWR0156
+U 1 1 5CFBC026
+P 10100 5100
+F 0 "#PWR0156" H 10100 4850 50  0001 C CNN
+F 1 "GND" H 10105 4927 50  0000 C CNN
+F 2 "" H 10100 5100 50  0001 C CNN
+F 3 "" H 10100 5100 50  0001 C CNN
+	1    10100 5100
+	1    0    0    -1
+$EndComp
+Wire Wire Line
+	10100 5100 10100 5050
+Wire Wire Line
+	10100 4750 10100 4700
+Connection ~ 10100 4400
+Wire Wire Line
+	10100 4400 10225 4400
 $EndSCHEMATC
