File: patch/patch.sch (KiCad schematic (older format))
At the start: 19 parts, among them IC1 LTC3261, J1 -5V, J2 5V, J3 GND, J4 Audio_IN, J5 S_B, J6 SAW, J7 S_A, U1 AD8611

Commit message: p2
Parts:
- added D1: LED, LEDs:LED_1206_HandSoldering, symbol Device:LED
- added R5: 2k2, Resistors_SMD:R_1206_HandSoldering, symbol Device:R
Connections:
- net -5V: now also D1.1 (K)
- net GND: now also R5.1
- new net: D1.2 (A), R5.2
Changed lines of the file:
@@
 	1    0    0    -1
 $EndComp
+$Comp
+L Device:R R5
+U 1 1 5CEFAE52
+P 2625 2900
+F 0 "R5" V 2418 2900 50  0000 C CNN
+F 1 "2k2" V 2509 2900 50  0000 C CNN
+F 2 "Resistors_SMD:R_1206_HandSoldering" V 2555 2900 50  0001 C CNN
+F 3 "~" H 2625 2900 50  0001 C CNN
+	1    2625 2900
+	-1   0    0    1
+$EndComp
+$Comp
+L power:GND #PWR0125
+U 1 1 5CEFB3E7
+P 2625 3100
+F 0 "#PWR0125" H 2625 2850 50  0001 C CNN
+F 1 "GND" H 2630 2927 50  0000 C CNN
+F 2 "" H 2625 3100 50  0001 C CNN
+F 3 "" H 2625 3100 50  0001 C CNN
+	1    2625 3100
+	1    0    0    -1
+$EndComp
+$Comp
+L power:-5V #PWR0126
+U 1 1 5CEFB757
+P 2625 2350
+F 0 "#PWR0126" H 2625 2450 50  0001 C CNN
+F 1 "-5V" H 2640 2523 50  0000 C CNN
+F 2 "" H 2625 2350 50  0001 C CNN
+F 3 "" H 2625 2350 50  0001 C CNN
+	1    2625 2350
+	1    0    0    -1
+$EndComp
+$Comp
+L Device:LED D1
+U 1 1 5CEFC0D8
+P 2625 2550
+F 0 "D1" V 2572 2628 50  0000 L CNN
+F 1 "LED" V 2663 2628 50  0000 L CNN
+F 2 "LEDs:LED_1206_HandSoldering" H 2625 2550 50  0001 C CNN
+F 3 "~" H 2625 2550 50  0001 C CNN
+	1    2625 2550
+	0    1    1    0
+$EndComp
+Wire Wire Line
+	2625 3100 2625 3050
+Wire Wire Line
+	2625 2700 2625 2750
+Wire Wire Line
+	2625 2400 2625 2350
 $EndSCHEMATC
